File: hardware/SomaAudio/SomaAudio.kicad_pcb (KiCad board)
At the start: 2 copper layers, 74 x 78.8 mm, 12 parts, among them CN1 0.1uF, CN2 0.1uF, IC1 DG406DJ, J3 Audio Out, U1 MCP23017_SP

Commit message: Checkpoint on hardware design
Parts:
- added C1: 0.1 uF, Capacitor_THT:C_Axial_L3.8mm_D2.6mm_P7.50mm_Horizontal, F.Cu at (126.0, 58.6)
- added C2: 0.1 uF, Capacitor_THT:C_Axial_L3.8mm_D2.6mm_P7.50mm_Horizontal, F.Cu at (126.8, 112.0)
- J5: renamed from Audio IN
- J6: renamed from AUDIO IN
- renumbered I2C to J17, GND to J2, VIN to J4
Connections:
- U1 pad 4: Net-(IC1-A3) -> Net-(IC1-EN)
- U1 pad 5: Net-(IC1-EN) -> Net-(IC1-A3)
Routing:
- net GND: track 231.9 -> 242.4 mm
- net VCC 5V: track 121.2 -> 128.5 mm
- net Net-(IC1-A3): track 33.2 -> 28.8 mm
- net Net-(J17-Pin_3): track 24.1 -> 26.5 mm
- net Net-(IC1-EN): track 37.7 -> 36.7 mm
