File: hardware/SomaAudio/SomaAudio.kicad_sch (KiCad schematic)
At the start: 12 parts, among them CN1 0.1uF, CN2 0.1uF, IC1 DG406DJ, J17 I2C, J2 Audio GND +, J3 Audio Out, J4 VIN, J5 Audio IN 1, J6 Audio IN 2, U1 MCP23017_SP

Commit message: Checkpoint on hardware design
Parts:
- added C1, C2: 0.1 uF, Capacitor_THT:C_Axial_L3.8mm_D2.6mm_P7.50mm_Horizontal, symbol Device:C
Connections:
- net GND: now also C1.1, C2.1
- net VCC 5V: now also C1.2, C2.2
- net at U1.4 (GPB3): now also IC1.18 (EN); no longer IC1.14 (A3)
- net at U1.5 (GPB4): now also IC1.14 (A3); no longer IC1.18 (EN)
