File: hardware/SomaButton/SomaButton.kicad_pcb (KiCad board)
At the start: 2 copper layers, 99.8 x 99.8 mm, 18 parts, among them J1 LED+, J2 LED GND, J3 BTN GND, J5 V12, J6 Buttons, J7 V5, U2 ULN2803A, U3 ULN2803A

Commit message: hardware: combo board, LED board, production outputs, arduino firmware
Co-Authored-By: Claude Opus 5.5 (1M context) <noreply@anthropic.com>
Parts:
- removed I2C: I2C, Connector_JST:JST_EH_S4B-EH_1x04_P2.50mm_Horizontal
- added J4: I2C, Connector_JST:JST_EH_S4B-EH_1x04_P2.50mm_Horizontal, F.Cu at (91.3, 51.8)
- turned R2 to 0 degrees
Connections:
- D3 pad 1: +VDC -> Net-(D3-K)
- D3 pad 2: Net-(D3-A) -> 3V3
- M1 pad 36: unconnected-(M1-3V3_OUT-Pad36) -> 3V3
- R1 pad 1: +VDC -> Net-(D3-K)
- R2 pad 1: +VDC -> Net-(D3-K)
Routing:
- net GND: track 185.2 -> 248.8 mm
- net 3V3: track 0.00 -> 49.9 mm, vias 0 -> 1
- net +VDC: track 55.6 -> 22.6 mm
- net Net-(J4-Pin_3): track 71.4 -> 49.0 mm, vias 2 -> 1
- net Net-(D3-A): track 18.8 -> 0.00 mm, vias 1 -> 0
- net Net-(J4-Pin_2): track 58.8 -> 74.3 mm, vias 1 -> 0
- net Net-(D3-K): track 0.00 -> 13.8 mm
- net Net-(J6-Pin_1): track 47.1 -> 44.6 mm
